File: clocking.kicad_sch (KiCad schematic)
At the start: 26 parts, among them IC1 LMV112SD_NOPB, J1 2337019-1, J2 2337019-1, U1 TXETALSANF-10.000000, U2 LDLN025M33R, U3 LDLN025M33R, U4 SN74LVC1G240DCKR

Commit message: Added PLL1, entered in MPNs of all parts
Parts:
- C1, C15, C16, C18, C19, C8: MPN (none) -> GRM1555C1E103JE01J; Manufacturer (none) -> Murata Electronics
- C10, C13, C17, C3, C6: MPN (none) -> GRM155R71C104KA88J; Manufacturer (none) -> Murata Electronics
- C11, C14, C4, C7: MPN (none) -> GRM1555C1H102JA01D; Manufacturer (none) -> Murata Electronics
- C12, C2, C5, C9: MPN (none) -> GRM155R70J105KA12J; Manufacturer (none) -> Murata Electronics
- IC1: MPN (none) -> LMV112SD/NOPB; Manufacturer (none) -> Texas Instruments; Manufacturer_Name Texas Instruments -> (none); Manufacturer_Part_Number LMV112SD/NOPB -> (none); Mouser Part Number 926-LMV112SD/NOPB -> (none); Mouser Price/Stock https://www.mouser.co.uk/ProductDetail/Texas-Instruments/LM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 -> (none)
- J1, J2: value 2337019-1 -> MMCX; MPN (none) -> 2337019-1; Manufacturer (none) -> TE Connectivity AMP Connectors
- U1: MPN (none) -> TXETALSANF-10.000000; Manufacturer (none) -> Taitien
- U2, U3: MF STMicroelectronics -> (none); MP LDLN025M33R -> (none); MPN (none) -> LDLN025M33R; Manufacturer (none) -> STMicroelectronics
- U4: MPN (none) -> SN74LVC1G240DCKR; Manufacturer (none) -> Texas Instruments
Connections:
- net EXT_REF_OUT: now reaches C15.1, IC1.6 (OUT_2)
- net EXT_REF renamed EXT_REF_IN_OUT
- net REF renamed REF_OUT
